Commit message: feat:add kdl_urdf_test.py

File: model/so_arm100_description/so100.urdf (robot description, URDF)
Before this commit: robot SO_5DOF_ARM100_8j_URDF.SLDASM, 9 links, 8 joints
Links:
- removed link Fixed_Jaw_tip
- removed link Moving_Jaw
- removed link Moving_Jaw_tip
- added link Moving Jaw, mass 0.0202443794940372; collision mesh filename=package://SO_5DOF_ARM100_8j_URDF.SLDASM/meshes/Moving Jaw.S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; visual mesh filename=package://SO_5DOF_ARM100_8j_URDF.SLDASM/meshes/Moving Jaw.S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
- link Base: geometry collision mesh filename=package://SO_5DOF_ARM100_8j_URDF.SLDASM/meshes/Base.STL; visual mesh filename=package://SO_5DOF_ARM100_8j_URDF.SLDASM/meshes/Base.STL
- link Fixed_Jaw: geometry collision mesh filename=package://SO_5DOF_ARM100_8j_URDF.SLDASM/meshes/Fixed_Jaw.STL; visual mesh filename=package://SO_5DOF_ARM100_8j_URDF.SLDASM/meshes/Fixed_Jaw.STL
- link Lower_Arm: geometry collision mesh filename=package://SO_5DOF_ARM100_8j_URDF.SLDASM/meshes/Lower_Arm.STL; visual mesh filename=package://SO_5DOF_ARM100_8j_URDF.SLDASM/meshes/Lower_Arm.STL
- link Rotation_Pitch: geometry collision mesh filename=package://SO_5DOF_ARM100_8j_URDF.SLDASM/meshes/Rotation_Pit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; visual mesh filename=package://SO_5DOF_ARM100_8j_URDF.SLDASM/meshes/Rotation_Pit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
- link Upper_Arm: geometry collision mesh filename=package://SO_5DOF_ARM100_8j_URDF.SLDASM/meshes/Upper_Arm.STL; visual mesh filename=package://SO_5DOF_ARM100_8j_URDF.SLDASM/meshes/Upper_Arm.STL
- link Wrist_Pitch_Roll: geometry collision mesh filename=package://SO_5DOF_ARM100_8j_URDF.SLDASM/meshes/Wrist_Pitch_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; visual mesh filename=package://SO_5DOF_ARM100_8j_URDF.SLDASM/meshes/Wrist_Pitch_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
Joints:
- removed joint Fixed_Jaw_tip_joint
- removed joint Moving_Jaw_tip_joint
- joint Elbow: limit lower=-0.2 upper=3.14159 effort=0 velocity=0 -> (none); origin xyz=0 0.11257 0.028 rpy=-1.5708 0 0 -> xyz=0 0.11257 0.028 rpy=0 0 0; type revolute -> continuous
- joint Jaw: child Moving_Jaw -> Moving Jaw; limit lower=0 upper=1.7 effort=0 velocity=0 -> (none); origin xyz=-0.0202 -0.0244 0 rpy=3.1416 0 3.33 -> xyz=-0.0202 -0.0244 0 rpy=3.1416 0 3.1416; type revolute -> continuous
- joint Pitch: axis -1 0 0 -> 1 0 0; limit lower=-0.1 upper=3.45 effort=0 velocity=0 -> (none); origin xyz=0 0.1025 0.0306 rpy=1.5708 0 0 -> xyz=0 0.1025 0.0306 rpy=0 0 0; type revolute -> continuous
- joint Rotation: axis 0 -1 0 -> 0 1 0; limit lower=-2.1 upper=2.1 effort=0 velocity=0 -> (none); type revolute -> continuous
- joint Wrist_Pitch: limit lower=-1.8 upper=1.8 effort=0 velocity=0 -> (none); origin xyz=0 0.0052 0.1349 rpy=-1.5708 0 0 -> xyz=0 0.0052 0.1349 rpy=0 0 0; type revolute -> continuous
- joint Wrist_Roll: axis 0 -1 0 -> 0 1 0; limit lower=-3.14159 upper=3.14159 effort=0 velocity=0 -> (none); origin xyz=0 -0.0601 0 rpy=0 1.5708 0 -> xyz=0 -0.0601 0 rpy=0 0 0; type revolute -> continuous
